File: EFM8_Tag-Connect/EFM8_Tag-Connect.sch (EAGLE design)
At the start: 10 parts, among them J1 MF-CON-2.54mm-01x08, J2 MF-CON-2.54mm-01x07, U1 EFM8BB10F2G-A-QFN20

Commit message: Finished EFM8 board.
Parts:
- C1: device MF_Passives:CAPACITOR_NP_0603 -> MF_Passives:CAPACITOR_NP_0402; MPN MF-CAP-0603-1uF -> MF-CAP-0402-1uF
- C2: device MF_Passives:CAPACITOR_NP_0603 -> MF_Passives:CAPACITOR_NP_0402; MPN MF-CAP-0603-0.1uF -> MF-CAP-0402-0.1uF
- J1: value MF-CON-2.54mm-01x08 -> MF-CON-2.54mm-01x10; device MF_Connectors:CON_01X08_PTH_2.54MM -> MF_Connectors:CON_01X10_PTH_2.54MM
- J2: value MF-CON-2.54mm-01x07 -> MF-CON-2.54mm-01x09; device MF_Connectors:CON_01X07_PTH_2.54MM -> MF_Connectors:CON_01X09_PTH_2.54MM
- R1: device MF_Passives:RESISTOR_0603 -> MF_Passives:RESISTOR_0402; MPN MF-RES-0603-10K -> MF-RES-0402-10K
- R2: device MF_Passives:RESISTOR_0603 -> MF_Passives:RESISTOR_0402; MPN MF-RES-0603-360 -> MF-RES-0402-360
Connections:
- net !RST!/C2CK: now also J2.PIN8
- net 3.3V: now also J1.PIN1
- net C2D: now also J2.PIN9
- net GND: now also J1.PIN2
- net P0.0: now also J1.PIN3; no longer D1.ANODE, J1.PIN1
- net P0.1: now also J1.PIN4; no longer J1.PIN2
- net P0.2: now also J1.PIN5; no longer J1.PIN3
- net P0.3: now also J1.PIN6; no longer J1.PIN4
- net P0.4: now also J1.PIN7; no longer J1.PIN5
- net P0.5: now also J1.PIN8; no longer J1.PIN6
- net P0.6: now also J1.PIN9; no longer J1.PIN7
- net P0.7: now also J1.PIN10; no longer J1.PIN8
- net P1.0: now also D1.ANODE
Changed lines of the file:
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@@
 <?xml version="1.0" encoding="utf-8"?>
 <!DOCTYPE eagle SYSTEM "eagle.dtd">
-<eagle version="7.4.0">
+<eagle version="7.6.0">
 <drawing>
 <settings>
@@
 </part>
 <part name="TC1" library="MF_Connectors" deviceset="CON_02X03" device="_TC2030-IDC" technology="_SILABS2TC" value="TC2030-IDC"/>
-<part name="C1" library="MF_Passives" deviceset="CAPACITOR_NP" device="_0603" value="1uF">
-<attribute name="MPN" value="MF-CAP-0603-1uF"/>
-</part>
-<part name="C2" library="MF_Passives" deviceset="CAPACITOR_NP" device="_0603" value="0.1uF">
-<attribute name="MPN" value="MF-CAP-0603-0.1uF"/>
-</part>
-<part name="R1" library="MF_Passives" deviceset="RESISTOR" device="_0603" value="10K">
-<attribute name="MPN" value="MF-RES-0603-10K"/>
+<part name="C1" library="MF_Passives" deviceset="CAPACITOR_NP" device="_0402" value="1uF">
+<attribute name="MPN" value="MF-CAP-0402-1uF"/>
+</part>
+<part name="C2" library="MF_Passives" deviceset="CAPACITOR_NP" device="_0402" value="0.1uF">
+<attribute name="MPN" value="MF-CAP-0402-0.1uF"/>
+</part>
+<part name="R1" library="MF_Passives" deviceset="RESISTOR" device="_0402" value="10K">
+<attribute name="MPN" value="MF-RES-0402-10K"/>
 </part>
 <part name="U$1" library="MF_Aesthetics" deviceset="GND_RAIL" device=""/>
@@
 </part>
 <part name="D1" library="MF_LEDs" deviceset="LED_SINGLE" device="-0603-RED" value="MF-LED-0603-RED"/>
-<part name="R2" library="MF_Passives" deviceset="RESISTOR" device="_0603" value="360">
-<attribute name="MPN" value="MF-RES-0603-360"/>
+<part name="R2" library="MF_Passives" deviceset="RESISTOR" device="_0402" value="360">
+<attribute name="MPN" value="MF-RES-0402-360"/>
 </part>
 <part name="U$5" library="MF_Aesthetics" deviceset="GND_RAIL" device=""/>
-<part name="J1" library="MF_Connectors" deviceset="CON_01X08" device="_PTH_2.54MM" value="MF-CON-2.54mm-01x08"/>
-<part name="J2" library="MF_Connectors" deviceset="CON_01X07" device="_PTH_2.54MM" value="MF-CON-2.54mm-01x07"/>
+<part name="J2" library="MF_Connectors" deviceset="CON_01X09" device="_PTH_2.54MM" value="MF-CON-2.54mm-01x09"/>
+<part name="J1" library="MF_Connectors" deviceset="CON_01X10" device="_PTH_2.54MM" value="MF-CON-2.54mm-01x10"/>
 </parts>
 <sheets>
@@
 <instance part="R2" gate="G$1" x="109.22" y="20.32" rot="R90"/>
 <instance part="U$5" gate="G$1" x="116.84" y="12.7"/>
-<instance part="J1" gate="G$1" x="99.06" y="88.9"/>
 <instance part="J2" gate="G$1" x="99.06" y="63.5"/>
+<instance part="J1" gate="G$1" x="99.06" y="93.98"/>
 </instances>
 <busses>
@@
 <wire x1="114.3" y1="20.32" x2="116.84" y2="20.32" width="0.1524" layer="91"/>
 <wire x1="116.84" y1="20.32" x2="116.84" y2="15.24" width="0.1524" layer="91"/>
+</segment>
+<segment>
+<pinref part="J1" gate="G$1" pin="PIN2"/>
+<wire x1="96.52" y1="91.44" x2="86.36" y2="91.44" width="0.1524" layer="91"/>
+<label x="88.9" y="91.44" size="1.016" layer="95" font="vector"/>
 </segment>
 </net>
@@
 <label x="60.96" y="20.32" size="1.016" layer="95" font="vector"/>
 </segment>
+<segment>
+<pinref part="J1" gate="G$1" pin="PIN1"/>
+<wire x1="86.36" y1="93.98" x2="96.52" y2="93.98" width="0.1524" layer="91"/>
+<label x="88.9" y="93.98" size="1.016" layer="95" font="vector"/>
+</segment>
 </net>
 <net name="!RST!/C2CK" class="0">
@@
 <label x="40.64" y="78.74" size="1.016" layer="95" font="vector"/>
 </segment>
+<segment>
+<pinref part="J2" gate="G$1" pin="PIN8"/>
+<wire x1="96.52" y1="45.72" x2="86.36" y2="45.72" width="0.1524" layer="91"/>
+<label x="88.9" y="45.72" size="1.016" layer="95" font="vector"/>
+</segment>
 </net>
 <net name="C2D" class="0">
@@
 <label x="73.66" y="45.72" size="1.016" layer="95" font="vector"/>
 </segment>
+<segment>
+<pinref part="J2" gate="G$1" pin="PIN9"/>
+<wire x1="96.52" y1="43.18" x2="86.36" y2="43.18" width="0.1524" layer="91"/>
+<label x="88.9" y="43.18" size="1.016" layer="95" font="vector"/>
+</segment>
 </net>
 <net name="P0.0" class="0">
@@
 <label x="73.66" y="88.9" size="1.016" layer="95" font="vector"/>
 <wire x1="71.12" y1="88.9" x2="96.52" y2="88.9" width="0.1524" layer="91"/>
-<pinref part="J1" gate="G$1" pin="PIN1"/>
-</segment>
-<segment>
-<pinref part="D1" gate="G$1" pin="ANODE"/>
-<wire x1="96.52" y1="20.32" x2="88.9" y2="20.32" width="0.1524" layer="91"/>
-<label x="91.44" y="20.32" size="1.016" layer="95" font="vector"/>
+<pinref part="J1" gate="G$1" pin="PIN3"/>
 </segment>
 </net>
@@
 <label x="73.66" y="86.36" size="1.016" layer="95" font="vector"/>
 <wire x1="71.12" y1="86.36" x2="96.52" y2="86.36" width="0.1524" layer="91"/>
-<pinref part="J1" gate="G$1" pin="PIN2"/>
+<pinref part="J1" gate="G$1" pin="PIN4"/>
 </segment>
 </net>
@@
 <label x="73.66" y="81.28" size="1.016" layer="95" font="vector"/>
 <wire x1="96.52" y1="81.28" x2="71.12" y2="81.28" width="0.1524" layer="91"/>
-<pinref part="J1" gate="G$1" pin="PIN4"/>
+<pinref part="J1" gate="G$1" pin="PIN6"/>
 </segment>
 </net>
@@
 <label x="73.66" y="83.82" size="1.016" layer="95" font="vector"/>
 <wire x1="71.12" y1="83.82" x2="96.52" y2="83.82" width="0.1524" layer="91"/>
-<pinref part="J1" gate="G$1" pin="PIN3"/>
+<pinref part="J1" gate="G$1" pin="PIN5"/>
 </segment>
 </net>
@@
 <label x="73.66" y="78.74" size="1.016" layer="95" font="vector"/>
 <wire x1="71.12" y1="78.74" x2="96.52" y2="78.74" width="0.1524" layer="91"/>
-<pinref part="J1" gate="G$1" pin="PIN5"/>
+<pinref part="J1" gate="G$1" pin="PIN7"/>
 </segment>
 </net>
@@
 <label x="73.66" y="76.2" size="1.016" layer="95" font="vector"/>
 <wire x1="96.52" y1="76.2" x2="71.12" y2="76.2" width="0.1524" layer="91"/>
-<pinref part="J1" gate="G$1" pin="PIN6"/>
+<pinref part="J1" gate="G$1" pin="PIN8"/>
 </segment>
 </net>
@@
 <label x="73.66" y="73.66" size="1.016" layer="95" font="vector"/>
 <wire x1="71.12" y1="73.66" x2="96.52" y2="73.66" width="0.1524" layer="91"/>
-<pinref part="J1" gate="G$1" pin="PIN7"/>
+<pinref part="J1" gate="G$1" pin="PIN9"/>
 </segment>
 </net>
@@
 <label x="73.66" y="71.12" size="1.016" layer="95" font="vector"/>
 <wire x1="71.12" y1="71.12" x2="96.52" y2="71.12" width="0.1524" layer="91"/>
-<pinref part="J1" gate="G$1" pin="PIN8"/>
+<pinref part="J1" gate="G$1" pin="PIN10"/>
 </segment>
 </net>
@@
 <pinref part="J2" gate="G$1" pin="PIN1"/>
 </segment>
-</net>
+<segment>
+<pinref part="D1" gate="G$1" pin="ANODE"/>
+<wire x1="96.52" y1="20.32" x2="88.9" y2="20.32" width="0.1524" layer="91"/>
+<label x="91.44" y="20.32" size="1.016" layer="95" font="vector"/>
+</segment>
+</net>

Commit message: Updated to recent library changes.
Parts:
- U1: value EFM8BB10F2G-A-QFN20 -> (none)
Changed lines of the file:
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@@
 <?xml version="1.0" encoding="utf-8"?>
 <!DOCTYPE eagle SYSTEM "eagle.dtd">
-<eagle version="7.6.0">
+<eagle version="7.4.0">
 <drawing>
 <settings>
@@
 </classes>
 <parts>
-<part name="U1" library="MF_IC_Digital" deviceset="EFM8BB10F(2/4/8)G-A-QFN20" device="" value="EFM8BB10F2G-A-QFN20">
+<part name="U1" library="MF_IC_Digital" deviceset="EFM8BB10F(2/4/8)G-A-QFN20" device="">
 <attribute name="MPN" value="EFM8BB10F2G-A-QFN20"/>
 </part>
