File: AVRISP2TC/AVRISP2TC.brd (EAGLE design)
At the start: 39.4 x 34 mm, 14 parts, among them U1 NCP1117LPST33T3G

Commit message: Major revamp of repo.
Changed lines of the file:
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@@
 <?xml version="1.0" encoding="utf-8"?>
 <!DOCTYPE eagle SYSTEM "eagle.dtd">
-<eagle version="7.6.0">
+<eagle version="7.4.0">
 <drawing>
 <settings>
@@
 </element>
 <element name="U1" library="MF_IC_Power" package="SOT-223-3" value="NCP1117LPST33T3G" x="28.575" y="28.575" smashed="yes" rot="R180">
-<attribute name="NAME" x="30.809" y="23.821" size="1.27" layer="25" font="vector" ratio="16" rot="R180"/>
+<attribute name="NAME" x="22.661" y="28.269" size="1.27" layer="25" font="vector" ratio="16" rot="R270"/>
 <attribute name="MPN" value="NCP1117LPST33T3G" x="28.575" y="28.575" size="1.778" layer="27" rot="R180" display="off"/>
 <attribute name="HOUSEPART" value="NO" x="28.575" y="28.575" size="1.778" layer="27" rot="R180" display="off"/>
@@
 <attribute name="VALUE" value="30306-6002HB" x="14.986" y="10.795" size="1.778" layer="27" rot="R270" display="off"/>
 <attribute name="NAME" x="20.478" y="12.827" size="0.8128" layer="25" font="vector" ratio="16" rot="R90"/>
+<attribute name="URL" value="" x="14.986" y="10.795" size="1.778" layer="27" rot="R270" display="off"/>
+<attribute name="HOUSEPART" value="" x="14.986" y="10.795" size="1.778" layer="27" rot="R270" display="off"/>
 </element>
 <element name="TC2030" library="PP_Connectors" package="30306-6002HB" value="30306-6002HB" x="33.655" y="10.795" rot="R270">
@@
 <attribute name="LABEL01" value="MISO" x="33.655" y="10.795" size="1.778" layer="27" rot="R270" display="off"/>
 <attribute name="VALUE" value="30306-6002HB" x="33.655" y="10.795" size="1.778" layer="27" rot="R270" display="off"/>
+<attribute name="URL" value="" x="33.655" y="10.795" size="1.778" layer="27" rot="R270" display="off"/>
+<attribute name="HOUSEPART" value="" x="33.655" y="10.795" size="1.778" layer="27" rot="R270" display="off"/>
 </element>
 <element name="10PIN_ISP" library="PP_Connectors" package="5103308-1" value="5103308-1" x="5.08" y="10.795" smashed="yes" rot="R270">
@@
 <attribute name="POPULATE" value="1" x="5.08" y="10.795" size="1.778" layer="27" rot="R270" display="off"/>
 <attribute name="NAME" x="0.635" y="21.336" size="0.8128" layer="25" font="vector" ratio="16"/>
+<attribute name="URL" value="" x="5.08" y="10.795" size="1.778" layer="27" rot="R270" display="off"/>
+<attribute name="HOUSEPART" value="" x="5.08" y="10.795" size="1.778" layer="27" rot="R270" display="off"/>
 </element>
 </elements>

Commit message: Fixed MISO/MOSI swap on 10Pin ISP header.
Connections:
- net MISO: now also 10PIN_ISP.9; no longer 10PIN_ISP.1
- net MOSI: now also 10PIN_ISP.1; no longer 10PIN_ISP.9
Routing:
- net MISO: track 33.2 -> 42.9 mm
Changed lines of the file:
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@@
 <layer number="44" name="Drills" color="7" fill="1" visible="no" active="yes"/>
 <layer number="45" name="Holes" color="7" fill="1" visible="no" active="yes"/>
-<layer number="46" name="Milling" color="3" fill="1" visible="no" active="yes"/>
+<layer number="46" name="Milling" color="3" fill="1" visible="yes" active="yes"/>
 <layer number="47" name="Measures" color="7" fill="1" visible="no" active="yes"/>
 <layer number="48" name="Document" color="7" fill="1" visible="yes" active="yes"/>
@@
 <element name="FRAME1" library="MF_Aesthetics" package="MF_FRAME_DEFAULT" value="" x="10.16" y="25.146">
 <attribute name="DNAME" value="Parker Dillmann" x="10.16" y="25.146" size="1.778" layer="27" display="off"/>
-<attribute name="REVNUM" value="REV: 1" x="10.16" y="25.146" size="1.778" layer="27" display="off"/>
+<attribute name="REVNUM" value="REV: 2" x="10.16" y="25.146" size="1.778" layer="27" display="off"/>
 <attribute name="MPN" value="" x="10.16" y="25.146" size="1.778" layer="27" display="off"/>
 <attribute name="HOUSEPART" value="0" x="10.16" y="25.146" size="1.778" layer="27" display="off"/>
@@
 <contactref element="6PIN_ISP" pad="1"/>
 <contactref element="TC2030" pad="1"/>
-<contactref element="10PIN_ISP" pad="1"/>
-<wire x1="6.35" y1="5.715" x2="15.748" y2="5.715" width="0.254" layer="1"/>
 <wire x1="16.256" y1="5.715" x2="34.163" y2="5.715" width="0.254" layer="1"/>
 <wire x1="34.163" y1="5.715" x2="34.925" y2="6.477" width="0.254" layer="1"/>
 <wire x1="34.925" y1="6.477" x2="34.925" y2="8.255" width="0.254" layer="1"/>
 <wire x1="16.256" y1="8.255" x2="16.256" y2="5.715" width="0.254" layer="1"/>
-<wire x1="16.256" y1="5.715" x2="15.748" y2="5.715" width="0.254" layer="1"/>
+<contactref element="10PIN_ISP" pad="9"/>
+<wire x1="6.35" y1="15.875" x2="16.637" y2="15.875" width="0.254" layer="16"/>
+<wire x1="16.637" y1="15.875" x2="18.542" y2="13.97" width="0.254" layer="16"/>
+<wire x1="18.542" y1="13.97" x2="18.542" y2="10.541" width="0.254" layer="16"/>
+<wire x1="18.542" y1="10.541" x2="16.256" y2="8.255" width="0.254" layer="16"/>
 </signal>
 <signal name="SCK">
@@
 <contactref element="TC2030" pad="4"/>
 <contactref element="6PIN_ISP" pad="4"/>
-<contactref element="10PIN_ISP" pad="9"/>
-<wire x1="6.35" y1="15.875" x2="7.239" y2="15.875" width="0.254" layer="1"/>
-<wire x1="7.239" y1="15.875" x2="12.319" y2="10.795" width="0.254" layer="1"/>
-<wire x1="12.319" y1="10.795" x2="13.716" y2="10.795" width="0.254" layer="1"/>
 <wire x1="13.716" y1="10.795" x2="13.716" y2="11.684" width="0.254" layer="1"/>
 <wire x1="13.716" y1="11.684" x2="13.97" y2="11.938" width="0.254" layer="1"/>
@@
 <wire x1="36.068" y1="9.652" x2="33.528" y2="9.652" width="0.254" layer="1"/>
 <wire x1="33.528" y1="9.652" x2="32.385" y2="10.795" width="0.254" layer="1"/>
+<contactref element="10PIN_ISP" pad="1"/>
+<wire x1="6.35" y1="5.715" x2="8.636" y2="5.715" width="0.254" layer="16"/>
+<wire x1="8.636" y1="5.715" x2="13.716" y2="10.795" width="0.254" layer="16"/>
 </signal>
 </signals>
