File: Macro_Duino/Macro_Duino.sch (EAGLE design)
At the start: 21 parts, among them J2 KLDX-0202-A, U1 ATMEGA328P-AU, X1 ABMM-16.000MHZ-B2-T

Commit message: Almost done with Macro Duino
Parts:
- removed J2: KLDX-0202-A, MF_Connectors:DC_PWR_JACK_2.0MM_RIGHT
- added C10, C9: 47pF, MF_Passives:CAPACITOR_NP_0603
- added C11, C13, C14, C17, C18, C22, C23: 0.1uF, MF_Passives:CAPACITOR_NP_0603
- added C12: 1uF, MF_Passives:CAPACITOR_NP_0603
- added C15, C16, C20, C21: 10uF, MF_Passives:CAPACITOR_NP_1206
- added C19: MF-CAP-4MM-10uF, MF_Passives:CAPACITOR_P_4MM
- added D2, D3: MF-LED-0805-RED, MF_LEDs:LED_SINGLE-0805-RED
- added FRAME1: MF_FRAMEDEFAULT, MF_Aesthetics:MF_FRAMEDEFAULT
- added ISP: MF-CON-2.54mm-2x3, MF_Connectors:CON_02X03_PTH_2.54MM
- added L1, L2: MI0603K300R-10, MF_Passives:INDUCTOR_0603
- added PWR_IN: KLDX-0202-A, MF_Connectors:DC_PWR_JACK_2.0MM_RIGHT
- added PW_SEL: MF-CON-2.54mm-01x03, MF_Connectors:CON_01X03_PTH_2.54MM
- added R10, R8: 360, MF_Passives:RESISTOR_0603
- added R11: 0, MF_Passives:RESISTOR_0603
- added R3: 5.1K, MF_Passives:RESISTOR_0603
- added R4, R5: 27, MF_Passives:RESISTOR_0603
- added R6, R9: 1K, MF_Passives:RESISTOR_0603
- added R7: 100K, MF_Passives:RESISTOR_0603
- added U$14: MF_LOGOLOGO_TEXT, PP_Aesthetics:MF_LOGOLOGO_TEXT
- added U$15: LHE_LOGOLHE_LOGO, PP_Aesthetics:LHE_LOGOLHE_LOGO
- added U2: FT230XQ-R, PP_DigitalIC:FT230XQ
- added U3: (no value), PP_DiscreteSemi:MOSFET_P-CHANNEL_SINGLE_SOT-23
- added U4: TPS2113ADRBR, PP_PowerIC:TPS211(2/3)ADR
- added U5: NCP1117LPST50T3G, MF_IC_Power:NCP1117LPST50T3G
- added U6: NCP1117LPST33T3G, MF_IC_Power:NCP1117LPST33T3G
- C1, C2: device MF_Passives:CAPACITOR_NP_0805 -> MF_Passives:CAPACITOR_NP_0603; MPN 08055A180JAT2A -> VJ0603A180JXACW1BC
- C3, C4, C5, C6, C8: device MF_Passives:CAPACITOR_NP_0805 -> MF_Passives:CAPACITOR_NP_0603; MPN MF-CAP-0805-0.1uF -> MF-CAP-0603-0.1uF
- J1: value (none) -> 105450-0101; MPN (none) -> 105450-0101
- R1: device MF_Passives:RESISTOR_0805 -> MF_Passives:RESISTOR_0603; MPN MF-RES-0805-10K -> MF-RES-0603-10K
- R2: device MF_Passives:RESISTOR_0805 -> MF_Passives:RESISTOR_0603; MPN MF-RES-0805-360 -> MF-RES-0603-360
- U1: value ATMEGA328P-AU -> ATMEGA328PB-AU; MPN (none) -> ATMEGA328PB-AU
Connections:
- removed net PD0: IOL.PIN8, U1.PD0
- removed net PD1: IOL.PIN7, U1.PD1
- new net 3V3OUT: C13.P$1, U2.3V3OUT
- new net CC1: J1.CC1, R3.P$1
- new net D+: R4.P$2, U2.USBDP
- new net D-: R5.P$2, U2.USBDM
- new net ILIM: R9.P$1, U4.ILIM
- new net N$1: D3.ANODE, R10.P$1
- new net N$3: R11.P$1, U4.OUT
- new net PW_EN: R6.P$2, U2.CBUS1
- new net PW_GT: R6.P$1, R7.P$1, U3.GATE
- new net RTS: C14.P$2, U2.RTS#
- new net RXD: IOL.PIN7, U1.PD1, U2.RXD
- new net TXD: IOL.PIN8, U1.PD0, U2.TXD
- new net TX_RX_LED: R8.P$1, U2.CBUS2
- new net TX_RX_LED_1: D2.ANODE, R8.P$2
- new net USB_5.0V_0: J1.VBUS, L1.P$1
- new net USB_5.0V_1: C11.P$1, C12.P$1, L1.P$2, R7.P$2, U2.VCC, U3.SOURCE
- new net USB_D+: C10.P$1, J1.D+, R4.P$1
- new net USB_D-: C9.P$1, J1.D-, R5.P$1
- new net USB_SHLD: J1.SHLD, L2.P$1
- new net USB_SW_5.0V: R10.P$2, U3.DRAIN, U4.IN2
- new net VCC: C3.P$1, C4.P$1, C5.P$1, C6.P$1, C7.P$1, ISP.PIN2, PW_SEL.PIN2, R1.P$1, TC1.PIN2, U1.AVCC, U1.VCC, U2.RESET#, U2.VCCIO
- new net VIN_5.0V: C16.P$1, C17.P$1, U4.IN1, U4.VSNS, U5.VOUT
- net 3.3V: now also C20.P$1, C23.P$1, PW_SEL.PIN1, U6.VOUT
- net 5.0V: now also C19.P$1, C21.P$1, C22.P$1, PW_SEL.PIN3, R11.P$2, U6.VIN; no longer C3.P$1, C4.P$1, C5.P$1, C6.P$1, C7.P$1, R1.P$1, TC1.PIN2, U1.AVCC, U1.VCC
- net GND: now also C10.P$2, C11.P$2, C12.P$2, C13.P$2, C15.P$2, C16.P$2, C17.P$2, C18.P$2, C19.P$2, C20.P$2, C21.P$2, C22.P$2, C23.P$2, C9.P$2, D1.CATHODE, D2.CATHODE, D3.CATHODE, ISP.PIN6, J1.GND, L2.P$2, PWR_IN.SLEEVE, PWR_IN.SLEEVE_SHUNT, R3.P$2, R9.P$2, U2.GND, U4.!EN, U4.GND, U5.GND/ADJ, U6.GND/ADJ; no longer R2.P$2
- net MISO: now also ISP.PIN1
- net MOSI: now also ISP.PIN4
- net N$2: now also D1.ANODE, R2.P$2; no longer D1.CATHODE, R2.P$1
- net RST: now also C14.P$1, ISP.PIN5
- net SCK: now also ISP.PIN3, R2.P$1; no longer D1.ANODE
- net VIN: now also C15.P$1, C18.P$1, PWR_IN.PIN, U5.VIN
Other:
- moved on the sheet: AD, D1, IOH, IOL, J1, POWER, R2

Commit message: Complete!~
Parts:
- removed PW_SEL: MF-CON-2.54mm-01x03, MF_Connectors:CON_01X03_PTH_2.54MM
- added JP1, JP2: 0, MF_Passives:RESISTOR_0805
- R11: device MF_Passives:RESISTOR_0603 -> MF_Passives:RESISTOR_0805; MPN MF-RES-0603-0 -> MF-RES-0805-0
- U$14: value MF_LOGOLOGO_TEXT -> MF_LOGOLOGO; device PP_Aesthetics:MF_LOGOLOGO_TEXT -> PP_Aesthetics:MF_LOGOLOGO
- U3: value (none) -> IRLML6401TRPBF
Connections:
- net 3.3V: now also JP2.P$1; no longer PW_SEL.PIN1
- net 5.0V: now also JP1.P$2; no longer PW_SEL.PIN3
- net VCC: now also JP1.P$1, JP2.P$2; no longer PW_SEL.PIN2

Commit message: Fixed FTDI power issue.
Parts:
- FRAME1: REVNUM REV: 1 -> REV: 2
- U3: value IRLML6401TRPBF -> IRLML6402TRPBF
Connections:
- removed net TX_RX_LED_1: D2.ANODE, R8.P$2
- new net N$4: D2.CATHODE, R8.P$2
- net 3V3OUT: now also C4.P$1, D2.ANODE, U2.RESET#, U2.VCCIO
- net GND: no longer D2.CATHODE
- net VCC: no longer C4.P$1, U2.RESET#, U2.VCCIO
Other:
- moved on the sheet: C4, D2, D3, R10, R6, R7, R8, U2, U3
