File: SWD2TC/SWD2TC.sch (EAGLE design)
At the start: 13 parts, among them J1 1761681-7, U1 NCP1117LPST33T3G

Commit message: Updating Readme and added files for SWD2TC
Parts:
- FRAME1: REVNUM REV: 2 -> REV: 1
Changed lines of the file:
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@@
 <part name="FRAME1" library="MF_Aesthetics" deviceset="MF_FRAME" device="DEFAULT" value="">
 <attribute name="DNAME" value="Parker Dillmann"/>
-<attribute name="REVNUM" value="REV: 2"/>
+<attribute name="REVNUM" value="REV: 1"/>
 </part>
 <part name="U$1" library="MF_Aesthetics" deviceset="GND_RAIL" device=""/>
