File: USB_Type-C_Projects/FTDI_FT230X_Example/FTDI_FT230X_Example.sch (EAGLE design)
At the start: 47 parts, among them J1 105450-0101, U1 FT230XQ-R, U135123 P8X32A-Q44, U2 IRLML6401TRPBF, U3 NCP1117LPST33T3G, U4 CAT24C512WI-GT3, X1 ABMM-6.000MHZ-B2-T

Commit message: Finished the FTDI_FT230X Example
Prop has been added and a header to monitor the current off the USB buss
Parts:
- removed 12351234152345, 1235235`, 235`5: 10K, PP_Passives:RESISTOR_0603
- removed 124121242, 12414124, 124235125, 12535, 1`21241: .1uF, PP_Passives:CAPACITOR_NON_POLAR_0603
- removed D1, D2, D3, D4: MF-LED-0603-RED, MF_LEDs:LED_SINGLE-0603-RED
- removed TP5: (no value), PP_Connectors:TEST_POINT_SINGLE_KEYSTONE_5115-5119
- removed U135123: P8X32A-Q44, PP_DigitalIC:P8X32A-Q44
- added BCD, TXRX, VBUS, VBUS_SW: MF-LED-0603-RED, MF_LEDs:LED_SINGLE-0603-RED
- added C10, C11, C13, C14, C15: .1uF, PP_Passives:CAPACITOR_NON_POLAR_0603
- added C16: 0.1uF, MF_Passives:CAPACITOR_NP_0603
- added J3: MF-CON-2.54mm-01x02, MF_Connectors:CON_01X02_PTH_2.54MM
- added J4, J6: MF-CON-2.54mm-01x05, MF_Connectors:CON_01X05_PTH_2.54MM
- added J5: MF-CON-2.54mm-01x03, MF_Connectors:CON_01X03_PTH_2.54MM
- added R10, R11, R12: 10K, PP_Passives:RESISTOR_0603
- added U5: P8X32A-Q44, PP_DigitalIC:P8X32A-Q44
- added U6: CAT24C512WI-GT3, PP_DigitalIC:EEPROM_I2CSOIC-8_W
- J2: value (none) -> MF-CON-2.54mm-01x03; device PP_Connectors:CON_01X08_2.54MM_PIN_HEADER -> MF_Connectors:CON_01X03_PTH_2.54MM; LABEL01 (none) -> P8; LABEL02 (none) -> P9; LABEL03 (none) -> P10; POPULATE (none) -> 0
- R6: value 150 -> 330
- TP1, TP2, TP3, TP4: value (none) -> 5115
- U2: value IRLML6401TRPBF -> IP4234CZ6,125; device PP_DiscreteSemi:MOSFET_P-CHANNEL_SINGLE_SOT-23 -> PP_Passives:IP4234CZ6
- U3: value NCP1117LPST33T3G -> IRLML6401TRPBF; device MF_IC_Power:NCP1117LPST33T3G -> PP_DiscreteSemi:MOSFET_P-CHANNEL_SINGLE_SOT-23
- U4: value CAT24C512WI-GT3 -> NCP1117LPST33T3G; device PP_DigitalIC:EEPROM_I2CSOIC-8_W -> MF_IC_Power:NCP1117LPST33T3G
Connections:
- net CC1/2 renamed CC1/1
- removed net N$1: D4.ANODE, R9.P$2
- removed net N$2: D1.ANODE, R6.P$2
- removed net N$41: R4.P$2, R5.P$1, U2.GATE
- removed net N$5: D2.ANODE, R7.P$2
- removed net N$6: D3.ANODE, R8.P$2
- new net N$10: R6.P$2, TXRX.ANODE
- new net N$11: R7.P$2, VBUS.ANODE
- new net N$12: R8.P$2, VBUS_SW.ANODE
- new net N$13: BCD.ANODE, R9.P$2
- new net N$14: C3.P$1, R3.P$1, U2.I/O2A
- new net N$15: C4.P$1, R2.P$1, U2.I/O2B
- new net N$8: R4.P$2, R5.P$1, U3.GATE
- new net SYSTEM_VBUS: C1.P$1, C2.P$1, J3.PIN2, R4.P$1, R6.P$1, R7.P$1, U1.VCC, U2.VB, U3.SOURCE
- net 3.3V: now also C10.2, C11.2, C13.2, C14.2, C15.2, R10.1, R11.2, R12.2, TP4.P$1, U4.VOUT, U5.VDD, U6.VCC; no longer 12351234152345.2, 1235235`.2, 124121242.2, 12414124.2, 124235125.2, 12535.2, 1`21241.2, 235`5.2, R6.P$1, TP5.P$1, U135123.VDD, U3.VOUT, U4.VCC
- net BCD_CHARGER: now also TP3.P$1; no longer TP4.P$1
- net D+: now also U2.I/O1A; no longer C3.P$1, R3.P$1
- net D-: now also U2.I/O1B; no longer C4.P$1, R2.P$1
- net GND: now also BCD.CATHODE, C10.1, C11.1, C13.1, C14.1, C15.1, TP1.P$1, U2.GND, U4.GND/ADJ, U5.!BOE, U5.VSS, U6.A0, U6.A1, U6.A2, U6.GND, U6.WP, VBUS.CATHODE, VBUS_SW.CATHODE; no longer 124121242.1, 12414124.1, 124235125.1, 12535.1, 1`21241.1, D2.CATHODE, D3.CATHODE, D4.CATHODE, TP2.P$1, U135123.!BOE, U135123.VSS, U3.GND/ADJ, U4.A0, U4.A1, U4.A2, U4.GND, U4.WP
- net P0: now also U5.P0; no longer U135123.P0
- net P1: now also U5.P1; no longer U135123.P1
- net P10: now also J2.PIN3, U5.P10; no longer U135123.P10
- net P11: now also J4.PIN1, U5.P11; no longer J2.1, U135123.P11
- net P12: now also J4.PIN2, U5.P12; no longer J2.2, U135123.P12
- net P13: now also J4.PIN3, U5.P13; no longer J2.3, U135123.P13
- net P14: now also J4.PIN4, U5.P14; no longer J2.4, U135123.P14
- net P15: now also J4.PIN5, U5.P15; no longer J2.5, U135123.P15
- net P16: now also J6.PIN1, U5.P16; no longer U135123.P16
- net P17: now also J6.PIN2, U5.P17; no longer U135123.P17
- net P18: now also J6.PIN3, U5.P18; no longer U135123.P18
- net P19: now also J6.PIN4, U5.P19; no longer U135123.P19
- net P2: now also U5.P2; no longer U135123.P2
- net P20: now also J6.PIN5, U5.P20; no longer U135123.P20
- net P21: now also J5.PIN1, U5.P21; no longer J2.6, U135123.P21
- net P22: now also J5.PIN2, U5.P22; no longer J2.7, U135123.P22
- net P23: now also J5.PIN3, U5.P23; no longer J2.8, U135123.P23
- net P24: now also U5.P24; no longer U135123.P24
- net P25: now also U5.P25; no longer U135123.P25
- net P26: now also U5.P26; no longer U135123.P26
- net P27: now also U5.P27; no longer U135123.P27
- net P3: now also U5.P3; no longer U135123.P3
- net P4: now also U5.P4; no longer U135123.P4
- net P5: now also U5.P5; no longer U135123.P5
- net P6: now also U5.P6; no longer U135123.P6
- net P7: now also U5.P7; no longer U135123.P7
- net P8: now also J2.PIN1, U5.P8; no longer U135123.P8
- net P9: now also J2.PIN2, U5.P9; no longer U135123.P9
- net RES: now also C16.P$2, R10.2, U5.!RES; no longer 12351234152345.1, U135123.!RES
- net RTS: now also C16.P$1
- net RX: now also U5.P30; no longer U135123.P30
- net SCL: now also R12.1, U5.P28, U6.SCL; no longer 235`5.1, U135123.P28, U4.SCL
- net SDA: now also R11.1, U5.P29, U6.SDA; no longer 1235235`.1, U135123.P29, U4.SDA
- net TX: now also U5.P31; no longer U135123.P31
- net TX_RX_LED: now also TXRX.CATHODE; no longer D1.CATHODE
- net USB_VBUS: now also J3.PIN1; no longer C1.P$1, C2.P$1, R4.P$1, R7.P$1, U1.VCC, U2.SOURCE
- net USB_VBUS_PORT: no longer TP1.P$1
- net USB_VBUS_SWITCHED: now also TP2.P$1, U3.DRAIN, U4.VIN; no longer TP3.P$1, U2.DRAIN, U3.VIN
- net X0: now also U5.X0; no longer U135123.X0
- net X1: now also U5.X1; no longer U135123.X1
Other:
- moved on the sheet: C1, C12, C2, C3, C4, C5, C6, C7, C8, C9, J1, L1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
