File: USB_Type-C_Projects/ATmega32u4_Example/ATmega32u4_Example.brd (EAGLE design)
At the start: 40.3 x 54.9 mm, 54 parts, among them J1 105450-0101, J2 282834-3, J3 282834-3, J4 MF-CON-2.54mm-01x11, J5 MF-CON-2.54mm-01x11, SW1 MF-SW-TACT-4.2MM, U1 IP4234CZ6,125, U2 ATMEGA32U4-AU, X1 ABM3B-16.000MHZ-D-1-X-T

Commit message: REV 2. Fixed USB ESD protection.
Routing:
- net 5V: track 246.2 -> 248.0 mm
Changed lines of the file:
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@@
 <?xml version="1.0" encoding="utf-8"?>
 <!DOCTYPE eagle SYSTEM "eagle.dtd">
-<eagle version="9.3.0">
+<eagle version="9.3.2">
 <drawing>
 <settings>
@@
 <attribute name="MPN" value="" x="10.16" y="8.128" size="1.778" layer="27" display="off"/>
 <attribute name="POPULATE" value="0" x="10.16" y="8.128" size="1.778" layer="27" display="off"/>
-<attribute name="REVNUM" value="REV: 1" x="10.16" y="3.048" size="0.8128" layer="21" font="vector" ratio="16"/>
+<attribute name="REVNUM" value="REV: 2" x="10.16" y="3.048" size="0.8128" layer="21" font="vector" ratio="16"/>
 <attribute name="URL" value="" x="10.16" y="8.128" size="1.778" layer="27" display="off"/>
 </element>
@@
 <via x="26.6675" y="45.593" extent="1-16" drill="0.254"/>
 <contactref element="U1" pad="3"/>
-<wire x1="26.6675" y1="45.593" x2="26.9175" y2="45.593" width="0.127" layer="1"/>
-<wire x1="26.9175" y1="45.593" x2="26.9175" y2="44.5745" width="0.127" layer="1"/>
+<wire x1="26.6675" y1="45.593" x2="26.9175" y2="45.343" width="0.127" layer="1"/>
+<wire x1="26.9175" y1="45.343" x2="26.9175" y2="44.5745" width="0.127" layer="1"/>
 </signal>
 <signal name="D-">
@@
 <wire x1="24.7675" y1="45.7835" x2="24.7675" y2="45.593" width="0.127" layer="16"/>
 <contactref element="U1" pad="4"/>
-<wire x1="24.7675" y1="45.593" x2="24.5175" y2="45.593" width="0.127" layer="1"/>
-<wire x1="24.5175" y1="45.593" x2="24.5175" y2="44.5745" width="0.127" layer="1"/>
+<wire x1="24.7675" y1="45.593" x2="24.5175" y2="45.343" width="0.127" layer="1"/>
+<wire x1="24.5175" y1="45.343" x2="24.5175" y2="44.5745" width="0.127" layer="1"/>
 </signal>
 <signal name="SHEILD1">
@@
 <wire x1="17.78" y1="35.814" x2="17.78" y2="35.052" width="0.254" layer="1"/>
 <via x="17.78" y="35.052" extent="1-16" drill="0.254"/>
-<wire x1="17.78" y1="35.052" x2="13.589" y2="39.243" width="0.254" layer="16"/>
-<wire x1="13.589" y1="39.243" x2="5.207" y2="39.243" width="0.254" layer="16"/>
 <wire x1="5.207" y1="39.243" x2="1.524" y2="39.243" width="0.254" layer="16"/>
 <wire x1="4.6355" y1="42.3545" x2="9.398" y2="47.117" width="0.254" layer="1"/>
@@
 <wire x1="14.351" y1="47.117" x2="11.777" y2="47.117" width="0.127" layer="1"/>
 <wire x1="11.777" y1="47.117" x2="11.286" y2="47.608" width="0.127" layer="1"/>
+<wire x1="16.637" y1="39.243" x2="17.78" y2="38.1" width="0.254" layer="16"/>
+<wire x1="17.78" y1="38.1" x2="17.78" y2="35.052" width="0.254" layer="16"/>
+<wire x1="5.207" y1="39.243" x2="16.637" y2="39.243" width="0.254" layer="16"/>
 </signal>
 <signal name="A0">

Commit message: updated with two (2 :O ) CC resistors
Parts:
- added R19: 10K, MF_Passives:R0603
- R2: value 22 -> 5.1K
- R4: value 10K -> 22
- moved R4 18.3 mm to (26.7, 39.6), turned to 270 degrees
- moved R2 6.59 mm to (29.8, 43.8)
- moved R3 1.91 mm to (24.8, 39.6)
- moved L2 1.40 mm to (31.2, 43.8)
Connections:
- removed net CC1/1: J1.A5, J1.B5, R1.P$1
- new net CC1: J1.A5, R1.P$1
- new net CC2: J1.B5, R2.P$1
- net 5V: now also R19.P$1; no longer R4.P$1
- net DM: now also R3.P$1; no longer R2.P$1
- net DP: now also R4.P$1; no longer R3.P$1
- net GND: now also R2.P$2
- net N$1: now also R3.P$2; no longer R2.P$2
- net N$2: now also R4.P$2; no longer R3.P$2
- net RESET: now also R19.P$2; no longer R4.P$2
Routing:
- net CC1/1: track 8.48 -> 0.00 mm, vias 2 -> 0
- net CC2: track 0.00 -> 8.25 mm, vias 0 -> 2
- net CC1: track 0.00 -> 3.55 mm
